File: schematic/Buttons.kicad_sch (KiCad schematic)
At the start: 6 parts, among them U5 GPTS203211B, U6 GPTS203211B, U7 GPTS203211B, U9 MAX6818EAP_T

Commit message: Adding Revisions 2 and 3
Parts:
- renumbered U7 to U13, U9 to U8
