File: schematic/MCU.kicad_sch (KiCad schematic)
At the start: 13 parts, among them U15 STM32F767VGT6, U8 GPTS203211B

Commit message: Adding Revisions 2 and 3
Parts:
- renumbered C8 to C25, C7 to C26, C9 to C27, C11 to C28, C12 to C29, R7 to R16, R6 to R17, S2 to S3, U8 to U16
