File: schematic/USB.kicad_sch (KiCad schematic)
At the start: 23 parts, among them J1 USB4105-GF-A, J12 TS-102-G-A, J4 B2B-XH-A, Q1 DMP3099L-7, U12 TPS61202DRCT, U14 MAX1898EUB42_T

Commit message: Adding Revisions 2 and 3
Parts:
- renumbered R4 to R1, R5 to R2, R2 to R4, R1 to R5
