File: motor-flasher/SPItoCAN.kicad_sch (KiCad schematic)
At the start: 13 parts, among them J9 WJ500V-5.08-3P, SW2 SS12D07VG4NSGAPA, U21 MCP2515-I_SO, U22 ISO1050DUBR, Y3 CSTNE16M0V530000R0

Commit message: Pushing current changes
Parts:
- renumbered C36 to C31, C37 to C32, C38 to C33, C39 to C34, C40 to C35, J9 to J8, PS6 to PS5, R22 to R10, R23 to R21, SW2 to SW1, U21 to U19, U22 to U20, Y3 to Y2

Commit message: Starting layout
Parts:
- added C21: 100nF, Capacitor_SMD:C_0402_1005Metric, symbol Device:C
Connections:
- net +3.3V: now also C21.2
- net GND: now also C21.1
Changed lines of the file:
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@@
+	)
+	(junction
+		(at 93.98 52.07)
+		(diameter 0)
+		(color 0 0 0 0)
 	)
 	(junction
@@
 	(wire
 		(pts
+			(xy 93.98 59.69) (xy 93.98 60.96)
+		)
+		(stroke
+			(width 0)
+			(type default)
+		)
+	)
+	(wire
+		(pts
 			(xy 191.77 64.77) (xy 190.5 64.77)
 		)
@@
 	(wire
 		(pts
+			(xy 93.98 52.07) (xy 99.06 52.07)
+		)
+		(stroke
+			(width 0)
+			(type default)
+		)
+	)
+	(wire
+		(pts
 			(xy 194.31 49.53) (xy 199.39 49.53)
 		)
@@
 	(wire
 		(pts
-			(xy 81.28 52.07) (xy 99.06 52.07)
+			(xy 81.28 52.07) (xy 93.98 52.07)
 		)
 		(stroke
@@
 	)
 	(symbol
+		(lib_id "power:GND")
+		(at 93.98 60.96 0)
+		(unit 1)
+		(exclude_from_sim no)
+		(in_bom yes)
+		(on_board yes)
+		(dnp no)
+		(fields_autoplaced yes)
+		(property "Reference" "#PWR064"
+			(at 93.98 67.31 0)
+			(effects
+				(font
+					(size 1.27 1.27)
+				)
+				(hide yes)
+			)
+		)
+		(property "Value" "GND"
+			(at 93.98 66.04 0)
+			(effects
+				(font
+					(size 1.27 1.27)
+				)
+			)
+		)
+		(property "Footprint" ""
+			(at 93.98 60.96 0)
+			(effects
+				(font
+					(size 1.27 1.27)
+				)
+				(hide yes)
+			)
+		)
+		(property "Datasheet" ""
+			(at 93.98 60.96 0)
+			(effects
+				(font
+					(size 1.27 1.27)
+				)
+				(hide yes)
+			)
+		)
+		(property "Description" ""
+			(at 93.98 60.96 0)
+			(effects
+				(font
+					(size 1.27 1.27)
+				)
+				(hide yes)
+			)
+		)
+		(pin "1"
+		)
+		(instances
+			(project "motor-flasher"
+				(path "/011ae556-31c3-4ee2-a722-f56ffd3fdd08/e3301e22-c54d-4c6d-8201-ed1434ad4e7e"
+					(reference "#PWR064")
+					(unit 1)
+				)
+			)
+		)
+	)
+	(symbol
 		(lib_id "Device:R")
 		(at 22.86 55.88 0)
@@
 					(unit 1)
 				)
+			)
+		)
+	)
+	(symbol
+		(lib_id "Device:C")
+		(at 93.98 55.88 180)
+		(unit 1)
+		(exclude_from_sim no)
+		(in_bom yes)
+		(on_board yes)
+		(dnp no)
+		(property "Reference" "C21"
+			(at 91.44 53.34 0)
+			(effects
+				(font
+					(size 1.27 1.27)
+				)
+			)
+		)
+		(property "Value" "100nF"
+			(at 88.138 54.864 0)
+			(effects
+				(font
+					(size 1.27 1.27)
+				)
+			)
+		)
+		(property "Footprint" "Capacitor_SMD:C_0402_1005Metric"
+			(at 93.0148 52.07 0)
+			(effects
+				(font
+					(size 1.27 1.27)
+				)
+				(hide yes)
+			)
+		)
+		(property "Datasheet" "~"
+			(at 93.98 55.88 0)
+			(effects
+				(font
+					(size 1.27 1.27)
+				)
+				(hide yes)
+			)
+		)
+		(property "Description" ""
+			(at 93.98 55.88 0)
+			(effects
+				(font
+					(size 1.27 1.27)
+				)
+				(hide yes)
+			)
+		)
+		(pin "1"
+		)
+		(pin "2"
+		)
+		(instances
+			(project "motor-flasher"
+				(path "/011ae556-31c3-4ee2-a722-f56ffd3fdd08/e3301e22-c54d-4c6d-8201-ed1434ad4e7e"
+					(reference "C21")
+					(unit 1)
+				)

Commit message: Beginning Layout Process
Parts:
- removed R21: 120, Resistor_SMD:R_0402_1005Metric, symbol Device:R
- added R9: 120, Resistor_SMD:R_0402_1005Metric, symbol Device:R
- added SW3, SW4: SS12D07VG4NSGAPA, Motor-Flasher:SS12D07_CNK, symbol 2024-05-28_19-32-11:SS12D07VG4NSGAPA
- J8: footprint revparts2:CUI_TB006-508-03BE -> Motor-Flasher:CUI_TB006-508-03BE
- PS5: footprint relevantparts:CONV_RFM-0505S -> Motor-Flasher:CONV_RFM-0505S
- SW1: footprint revparts2:SS12D07_CNK -> Motor-Flasher:SS12D07_CNK
- U19: footprint revparts2:SOIC127P1030X265-18N -> Motor-Flasher:SOIC127P1030X265-18N
- U20: footprint revparts2:SOP254P1040X485-8N -> Motor-Flasher:SOP254P1040X485-8N
- Y2: footprint revparts2:OSC_CSTNE16M0V530000R0 -> Motor-Flasher:OSC_CSTNE16M0V530000R0
Connections:
- net CANL: now also R9.2
- net CAN_RX: now also SW4.1; no longer U20.2 (RXD)
- net CAN_TX: now also SW3.1; no longer U20.3 (TXD)
- net at SW1.2: now also R9.1
- new net CANRX: SW4.3
- new net CANRX_OUT: SW4.2, U20.2 (RXD)
- new net CANTX: SW3.3
- new net CANTX_OUT: SW3.2, U20.3 (TXD)
Other:
- moved on the sheet: C35, R10, SW1

Commit message: Removed ERC Errors and Warnings
Parts:
- removed C31, C32: 7pF, Capacitor_SMD:C_0603_1608Metric, symbol Device:C
- removed J8: WJ500V-5.08-3P, Motor-Flasher:CUI_TB006-508-03BE, symbol TB006-508-03BE:TB006-508-03BE
- removed PS5: B0505S-1WR3, Motor-Flasher:CONV_RFM-0505S, symbol RFM-0505S:RFM-0505S
- removed SW1, SW3, SW4: SS12D07VG4NSGAPA, Motor-Flasher:SS12D07_CNK, symbol 2024-05-28_19-32-11:SS12D07VG4NSGAPA
- removed U19: MCP2515-I_SO, Motor-Flasher:SOIC127P1030X265-18N, symbol MCP2515-I_SO:MCP2515-I_SO
- removed U20: ISO1050DUBR, Motor-Flasher:SOP254P1040X485-8N, symbol ISO1050DUBR:ISO1050DUBR
- added J3: WJ500V-5.08-3P, Motor-Flasher:CUI_TB006-508-03BE, symbol Motor_Flasher_Modified:TB006-508-03BE
- added PS1: B0505S-1WR3, Motor-Flasher:CONV_RFM-0505S, symbol Motor_Flasher_Modified:RFM-0505S
- added SW4: SS12D07VG4NSGAPA_120Ohms, Motor-Flasher:SS12D07_CNK, symbol Motor_Flasher_Modified:SS12D07VG4NSGAPA_120Ohms
- added SW6, SW7: SS12D07VG4NSGAPA, Motor-Flasher:SS12D07_CNK, symbol Motor_Flasher_Modified:SS12D07VG4NSGAPA_Signals
- added U5: MCP2515-I_SO, Motor-Flasher:SOIC127P1030X265-18N, symbol Motor_Flasher_Modified:MCP2515-I_SO
- added U6: ISO1050DUBR, Motor-Flasher:SOP254P1040X485-8N, symbol Motor_Flasher_Modified:ISO1050DUBR
Connections:
- net +3.3V: now also U5.18 (VDD), U6.1 (VCC1)
- net +5V: now also PS1.2 (+VIN)
- net CANH: now also J3.3, SW4.3, U6.7 (CANH)
- net CANL: now also J3.2, U6.6 (CANL)
- net CANRX: now also SW7.3
- net CANRX_OUT: now also SW7.2, U6.2 (RXD)
- net CANTX: now also SW6.3
- net CANTX_OUT: now also SW6.2, U6.3 (TXD)
- net CAN_GND: now also J3.1, PS1.3 (-VOUT), U6.5 (GND2)
- net CAN_RX: now also SW7.1, U5.2 (RXCAN)
- net CAN_TX: now also SW6.1, U5.1 (TXCAN)
- net CAN_VDD: now also PS1.4 (+VOUT), U6.8 (VCC2)
- net CS: now also U5.16 (~{CS})
- net GND: now also PS1.1 (-VIN), U5.9 (VSS), U6.4 (GND1)
- net INT: now also U5.12 (~{INT})
- net MISO: now also U5.15 (SO)
- net MOSI: now also U5.14 (SI)
- net OSC1: now also U5.8 (OSC1)
- net OSC2: now also U5.7 (OSC2)
- net SCK: now also U5.13 (SCK)
- net at R10.2: now also U5.17 (~{RESET})
- net at R9.1: now also SW4.2
