File: motor-flasher/MCU.kicad_sch (KiCad schematic)
At the start: 20 parts, among them J2 Conn_01x04_MountingPin, SW5 SS12D07VG4NSGAPA, U8 STM32F407VGT6, Y1 CSTNE16M0V530000R0

Commit message: Pushing current changes
Parts:
- added U10: STM32F405RGT6, STM32F405RGT6:QFP50P1200X1200X160-64N, symbol STM32F405RGT6:STM32F405RGT6
Changed lines of the file:
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@@
+	)
+	(symbol
+		(lib_id "STM32F405RGT6:STM32F405RGT6")
+		(at 198.12 158.75 0)
+		(unit 1)
+		(exclude_from_sim no)
+		(in_bom yes)
+		(on_board yes)
+		(dnp no)
+		(fields_autoplaced yes)
+		(property "Reference" "U10"
+			(at 198.12 95.25 0)
+			(effects
+				(font
+					(size 1.27 1.27)
+				)
+			)
+		)
+		(property "Value" "STM32F405RGT6"
+			(at 198.12 97.79 0)
+			(effects
+				(font
+					(size 1.27 1.27)
+				)
+			)
+		)
+		(property "Footprint" "STM32F405RGT6:QFP50P1200X1200X160-64N"
+			(at 198.12 158.75 0)
+			(effects
+				(font
+					(size 1.27 1.27)
+				)
+				(justify bottom)
+				(hide yes)
+			)
+		)
+		(property "Datasheet" ""
+			(at 198.12 158.75 0)
+			(effects
+				(font
+					(size 1.27 1.27)
+				)
+				(hide yes)
+			)
+		)
+		(property "Description" ""
+			(at 198.12 158.75 0)
+			(effects
+				(font
+					(size 1.27 1.27)
+				)
+				(hide yes)
+			)
+		)
+		(property "PARTREV" "LTR"
+			(at 198.12 158.75 0)
+			(effects
+				(font
+					(size 1.27 1.27)
+				)
+				(justify bottom)
+				(hide yes)
+			)
+		)
+		(property "STANDARD" "IPC-7351B"
+			(at 198.12 158.75 0)
+			(effects
+				(font
+					(size 1.27 1.27)
+				)
+				(justify bottom)
+				(hide yes)
+			)
+		)
+		(property "MANUFACTURER" "STMicroelectronics"
+			(at 198.12 158.75 0)
+			(effects
+				(font
+					(size 1.27 1.27)
+				)
+				(justify bottom)
+				(hide yes)
+			)
+		)
+		(pin "62"
+		)
+		(pin "4"
+		)
+		(pin "16"
+		)
+		(pin "25"
+		)
+		(pin "8"
+		)
+		(pin "51"
+		)
+		(pin "58"
+		)
+		(pin "7"
+		)
+		(pin "64"
+		)
+		(pin "63"
+		)
+		(pin "60"
+		)
+		(pin "9"
+		)
+		(pin "37"
+		)
+		(pin "43"
+		)
+		(pin "49"
+		)
+		(pin "48"
+		)
+		(pin "35"
+		)
+		(pin "41"
+		)
+		(pin "32"
+		)
+		(pin "61"
+		)
+		(pin "45"
+		)
+		(pin "33"
+		)
+		(pin "31"
+		)
+		(pin "40"
+		)
+		(pin "39"
+		)
+		(pin "46"
+		)
+		(pin "28"
+		)
+		(pin "56"
+		)
+		(pin "53"
+		)
+		(pin "18"
+		)
+		(pin "2"
+		)
+		(pin "36"
+		)
+		(pin "10"
+		)
+		(pin "54"
+		)
+		(pin "24"
+		)
+		(pin "57"
+		)
+		(pin "27"
+		)
+		(pin "21"
+		)
+		(pin "1"
+		)
+		(pin "20"
+		)
+		(pin "17"
+		)
+		(pin "22"
+		)
+		(pin "26"
+		)
+		(pin "11"
+		)
+		(pin "6"
+		)
+		(pin "42"
+		)
+		(pin "19"
+		)
+		(pin "30"
+		)
+		(pin "34"
+		)
+		(pin "55"
+		)
+		(pin "52"
+		)
+		(pin "50"
+		)
+		(pin "47"
+		)
+		(pin "23"
+		)
+		(pin "44"
+		)
+		(pin "5"
+		)
+		(pin "3"
+		)
+		(pin "29"
+		)
+		(pin "38"
+		)
+		(pin "59"
+		)
+		(pin "15"
+		)
+		(pin "12"
+		)
+		(pin "14"
+		)
+		(pin "13"
+		)
+		(instances
+			(project ""
+				(path "/011ae556-31c3-4ee2-a722-f56ffd3fdd08/21b9991f-ddde-447d-9f53-2b3773ea9e1b"
+					(reference "U10")
+					(unit 1)
+				)
+			)
+		)
 	)
 	(symbol

Commit message: Added Updates
Parts:
- removed J2: Conn_01x04_MountingPin, Connector_PinHeader_2.54mm:PinHeader_1x04_P2.54mm_Horizontal, symbol Connector_Generic_MountingPin:Conn_01x04_MountingPin
- added J2: Conn_01x05_Pin, symbol Connector:Conn_01x05_Pin
- added R24, R25, R26: 4.7k, Resistor_SMD:R_0402_1005Metric, symbol Device:R
Connections:
- net +3.3V: now also J2.5 (Pin_5), R24.1, R25.1, R26.1
- net GND: now also J2.3 (Pin_3)
- net I2C_SCL: now also U10.58 (PB6), R24.2
- net I2C_SDA: now also U10.59 (PB7), R25.2
- net LCD_INT: now also U10.61 (PB8), R26.2
- net NRST: now also J2.4 (Pin_4)
- net Sys_CLK: now also U10.49 (PA14/JTCK-SWCLK), J2.1 (Pin_1)
- net Sys_SDIO: now also U10.46 (PA13/JMS-SWDIO), J2.2 (Pin_2)
- no-connect marks 62 -> 61
Other:
- moved on the sheet: C18, C7, R16, R8, S10, SW5

Commit message: Starting layout
Parts:
- added C10, C22, C23, C24: 100nF, symbol Device:C
- added C8, C9: 2.2uF, Capacitor_SMD:C_0402_1005Metric, symbol Device:C
Connections:
- net +3.3V: now also U10.19 (VDD), U10.32 (VDD__1), U10.48 (VDD__2), U10.64 (VDD__3), C10.1, C22.1, C23.1, C24.1
- net Boot0: now also U10.60 (BOOT0)
- net GND: now also U10.18 (VSS), U10.63 (VSS__1), C10.2, C22.2, C23.2, C24.2, C8.2, C9.2
- net LCD_INT: now also U10.57 (PB5); no longer U10.61 (PB8)
- net NRST: now also U10.7 (NRST)
- net Osc1: now also U10.5 (PH0/OSC_IN)
- net Osc2: now also U10.6 (PH1/OSC_OUT)
- net at U10.31 (VCAP_1): now also C8.1
- net at U10.47 (VCAP_2): now also C9.1
- no-connect marks 61 -> 62

Commit message: Beginning Layout Process
Parts:
- removed C11, C12, C13, C15: 100nF, Capacitor_SMD:C_0402_1005Metric, symbol Device:C
- removed C16, C17: 2.2uF, Capacitor_SMD:C_0402_1005Metric, symbol Device:C
- removed R18, R19, R20: 4.7k, Resistor_SMD:R_0402_1005Metric, symbol Device:R
- removed U8: STM32F407VGT6, revparts2:QFP50P1600X1600X160-100N, symbol STM32F407VGT6:STM32F407VGT6
- added C25: 100nF, Capacitor_SMD:C_0402_1005Metric, symbol Device:C
- added R6: 2.5k, Resistor_SMD:R_0603_1608Metric, symbol Device:R
- C10, C22, C23, C24: footprint (none) -> Capacitor_SMD:C_0402_1005Metric
- C19, C20: value 30pF -> 7pF
- J2: value Conn_01x05_Pin -> CS-1109-1X5(L11.5)PA6T; footprint (none) -> Connector_PinHeader_2.54mm:PinHeader_1x05_P2.54mm_Horizontal
- S10: footprint revparts2:TS-1088-AR02016 -> Motor-Flasher:TS-1088-AR02016
- SW5: footprint revparts2:SS12D07_CNK -> Motor-Flasher:SOT95P275X110-6N
- U10: footprint STM32F405RGT6:QFP50P1200X1200X160-64N -> Motor-Flasher:QFP50P1200X1200X160-64N
- Y1: footprint RevParts:OSC_CSTNE16M0V530000R0 -> Motor-Flasher:OSC_CSTNE16M0V530000R0
Connections:
- net +3.3V: now also U10.1 (VBAT), U10.13 (VDDA), C25.1
- net Boot0: now also C7.1; no longer C7.2
- net CS1: now also U10.24 (PC4)
- net D+: now also U10.45 (PA12)
- net D-: now also U10.44 (PA11)
- net Deb_Down: now also U10.40 (PC9)
- net Deb_Up: now also U10.42 (PA9)
- net Deb_back: now also U10.8 (PC0)
- net Deb_select: now also U10.41 (PA8)
- net GND: now also C7.2, U10.12 (VSSA), C25.2, R6.2; no longer C7.1
- net INT1: now also U10.25 (PC5)
- net SPI_MISO: now also U10.22 (PA6/SPI1_MISO)
- net SPI_MOSI: now also U10.23 (PA7/SPI1_MOSI)
- net SPI_SCK: now also U10.21 (PA5/SPI1_SCK)
- net at U10.28 (PB2/BOOT1): now also R6.1
- net CAN_RX: now reaches U10.33 (PB12)
- net CAN_TX: now reaches U10.34 (PB13)
- no-connect marks 62 -> 30
Other:
- moved on the sheet: C10, C18, C19, C20, C22, C23, C24, C7, C9, J2, R16, R24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

Commit message: Removed ERC Errors and Warnings
Parts:
- removed C19, C20: 7pF, Capacitor_SMD:C_0402_1005Metric, symbol Device:C
- removed S10: TS-1088-AR02016, Motor-Flasher:TS-1088-AR02016, symbol dk_Pushbutton-Switches:GPTS203211B
- removed SW5: SS12D07VG4NSGAPA, Motor-Flasher:SOT95P275X110-6N, symbol 2024-05-28_19-32-11:SS12D07VG4NSGAPA
- removed U10: STM32F405RGT6, Motor-Flasher:QFP50P1200X1200X160-64N, symbol STM32F405RGT6:STM32F405RGT6
- added S1: TS-1088-AR02016, Motor-Flasher:TS-1088-AR02016, symbol Motor_Flasher_Modified:TS-1088-ARO2016_Mod
- added SW3: SS12D07VG4NSGAPA_Boot, Motor-Flasher:SOT95P275X110-6N, symbol Motor_Flasher_Modified:SS12D07VG4NSGAPA_Boot
- added U8: STM32F405RGT6, Motor-Flasher:QFP50P1200X1200X160-64N, symbol Motor_Flasher_Modified:STM32F405RGT6
Connections:
- net +3.3V: now also SW3.3, U8.1 (VBAT), U8.13 (VDDA), U8.19 (VDD), U8.32 (VDD__1), U8.48 (VDD__2), U8.64 (VDD__3)
- net Boot0: now also U8.60 (BOOT0)
- net CAN_RX: now also U8.33 (PB12)
- net CAN_TX: now also U8.34 (PB13)
- net CS1: now also U8.24 (PC4)
- net D+: now also U8.45 (PA12)
- net D-: now also U8.44 (PA11)
- net Deb_Down: now also U8.40 (PC9)
- net Deb_Up: now also U8.42 (PA9)
- net Deb_back: now also U8.8 (PC0)
- net Deb_select: now also U8.41 (PA8)
- net GND: now also S1.1, SW3.1, U8.12 (VSSA), U8.18 (VSS), U8.63 (VSS__1)
- net I2C_SCL: now also U8.58 (PB6)
- net I2C_SDA: now also U8.59 (PB7)
- net INT1: now also U8.25 (PC5)
- net NRST: now also U8.7 (NRST)
- net SPI_MISO: now also U8.22 (PA6/SPI1_MISO)
- net SPI_MOSI: now also U8.23 (PA7/SPI1_MOSI)
- net SPI_SCK: now also U8.21 (PA5/SPI1_SCK)
- net Sys_CLK: now also U8.49 (PA14/JTCK-SWCLK)
- net Sys_SDIO: now also U8.46 (PA13/JMS-SWDIO)
- net at R16.1: now also S1.2
- net at R6.1: now also U8.28 (PB2/BOOT1)
- net at C8.1: now also U8.31 (VCAP_1)
- net at C9.1: now also U8.47 (VCAP_2)
- net at R8.1: now also SW3.2
- net LCD_INT renamed LCD_Int
- net LCD_Int: now also U8.57 (PB5)
- net Osc1 renamed OscIn
- net OscIn: now also U8.5 (PH0/OSC_IN)
- net Osc2 renamed OscOut
- net OscOut: now also U8.6 (PH1/OSC_OUT)

Commit message: Rough Placement and Design
Parts:
- SW3: footprint Motor-Flasher:SOT95P275X110-6N -> Motor-Flasher:SS12D07_CNK
Changed lines of the file:
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@@
 		(on_board yes)
 		(dnp no)
-		(fields_autoplaced yes)
 		(property "Reference" "SW3"
 			(at 20.32 71.12 0)
@@
 		)
 		(property "Value" "SS12D07VG4NSGAPA_Boot"
-			(at 20.32 73.66 0)
+			(at 29.21 72.39 0)
 			(effects
 				(font
@@
 			)
 		)
-		(property "Footprint" "Motor-Flasher:SOT95P275X110-6N"
+		(property "Footprint" "Motor-Flasher:SS12D07_CNK"
 			(at 35.306 98.044 0)
 			(effects
