File: motor-flasher/Voltage Regulator.kicad_sch (KiCad schematic)
At the start: 3 parts, among them U3 LD1117S33TR

Commit message: Beginning Layout Process
Parts:
- U3: footprint revparts2:SOT230P700X180-4N -> Motor-Flasher:SOT230P700X180-4N
Connections:
- net VCC renamed Vout
Other:
- moved on the sheet: C1, C2

Commit message: Removed ERC Errors and Warnings
Parts:
- removed U3: LD1117S33TR, Motor-Flasher:SOT230P700X180-4N, symbol LD1117S33TR:LD1117S33TR
- added C3: 2.2uF, Capacitor_SMD:C_0402_1005Metric, symbol Device:C
- added C4: 47uF, Capacitor_SMD:C_0805_2012Metric, symbol Device:C
- added C5: 10uF, Capacitor_SMD:C_0805_2012Metric, symbol Device:C
- added C6: 100nF, Capacitor_SMD:C_0402_1005Metric, symbol Device:C
- added L1: 6.8uH, Motor-Flasher:CDRH5D28RHP, symbol Device:L
- added R3: 2.87M, Resistor_SMD:R_0805_2012Metric, symbol Device:R
- added R7: 390k, Resistor_SMD:R_0805_2012Metric, symbol Device:R
- added U10: LD1117S33TR, Motor-Flasher:SOT230P700X180-4N, symbol Motor_Flasher_Modified:LD1117S33TR
- added U3: TPS61027DRCR, Motor-Flasher:VREG_V62_16624-01YE, symbol Motor_Flasher_Modified:TPS61027DRCR
Connections:
- net +3.3V: now also U10.2 (OUT), U10.4 (OUT__1)
- net GND: now also C3.2, C4.2, C5.1, C6.1, R7.2, U10.1 (GND), U3.10 (PGND), U3.11 (EP), U3.5 (GND), U3.8 (PS)
- net Vout: now also C5.2, C6.2, L1.1, R3.1, U10.3 (IN), U3.1 (EN), U3.6 (VBAT)
- new net: L1.2, U3.9 (SW)
- new net +5V: C3.1, C4.1, U3.2 (VOUT)
- new net LBI: R3.2, R7.1, U3.7 (LBI)
- no-connect marks 0 -> 2
Other:
- moved on the sheet: C1, C2

Commit message: Rough Placement and Design
Parts:
- added TP4, TP5: TestPoint, symbol Connector:TestPoint
Connections:
- net +3.3V: now also TP4.1
- net +5V: now also TP5.1
