File: motor-flasher/motor-flasher.kicad_pcb (KiCad board)
At the start: 2 copper layers, 115.7 x 107.6 mm, 114 parts, among them J1 USB4105-GF-A, J10 WJ500V-5.08-3P, J11 WJ500V-5.08-3P, J12 TS-102-G-A, J2 Conn_01x04_MountingPin, J4 B2B-PH-K-S-GW, J8 WJ500V-5.08-3P, J9 WJ500V-5.08-3P, SW1 SS12D07VG4NSGAPA, SW2 SS12D07VG4NSGAPA, SW3 SS12D07VG4NSGAPA, SW4 SS12D07VG4NSGAPA, SW5 SS12D07VG4NSGAPA, U1 MAX16054AZT_T, U19 MCP2515-I_SO, U2 MAX16054AZT_T, U20 ISO1050DUBR, U21 MCP2515-I_SO, U22 ISO1050DUBR, U23 MCP2515-I_SO, U24 ISO1050DUBR, U25 MCP2515-I_SO, U26 ISO1050DUBR, U3 LD1117S33TR, U4 MAX16054AZT_T, U5 MAX16054AZT_T, U6 TPS61027DRCR, U7 BQ24075RGTT, U8 STM32F407VGT6, U9 PCF8574T_3_518, Y1 CSTNE16M0V530000R0, Y2 CSTNE16M0V530000R0, Y3 CSTNE16M0V530000R0, Y4 CSTNE16M0V530000R0, Y5 CSTNE16M0V530000R0

Commit message: Beginning Layout Process
Parts:
- removed C12, C13, C15, C38, C39, C40, C43, C44, C45, C48, C49, C50: 100nF, Capacitor_SMD:C_0402_1005Metric
- removed C16, C17: 2.2uF, Capacitor_SMD:C_0402_1005Metric
- removed C36, C37, C41, C42, C46, C47: 7pF, Capacitor_SMD:C_0603_1608Metric
- removed J10, J11, J9: WJ500V-5.08-3P, revparts2:CUI_TB006-508-03BE
- removed J12: TS-102-G-A, TS_102_G_A:SAMTEC_TS-102-G-A
- removed PS6, PS7, PS8: B0505S-1WR3, relevantparts:CONV_RFM-0505S
- removed R11, R12, R22: 10k, Resistor_SMD:R_0402_1005Metric
- removed R14: 1.18K, Resistor_SMD:R_0402_1005Metric
- removed R15: 25k, Resistor_SMD:R_0805_2012Metric
- removed R17: 1.5k, Resistor_SMD:R_0402_1005Metric
- removed R18, R19, R20: 4.7k, Resistor_SMD:R_0402_1005Metric
- removed R21, R23, R27: 120, Resistor_SMD:R_0402_1005Metric
- removed U21, U23, U25: MCP2515-I_SO, revparts2:SOIC127P1030X265-18N
- removed U22, U24, U26: ISO1050DUBR, revparts2:SOP254P1040X485-8N
- removed U7: BQ24075RGTT, revparts2:QFN50P300X300X100-17N
- removed U8: STM32F407VGT6, revparts2:QFP50P1600X1600X160-100N
- removed Y3, Y4, Y5: CSTNE16M0V530000R0, revparts2:OSC_CSTNE16M0V530000R0
- added C21: 100nF, Capacitor_SMD:C_0402_1005Metric, F.Cu at (225.2, 74.9)
- added C22: 100nF, Capacitor_SMD:C_0402_1005Metric, F.Cu at (-74.2, 170.5)
- added C23: 100nF, Capacitor_SMD:C_0402_1005Metric, F.Cu at (-74.2, 172.5)
- added C24: 100nF, Capacitor_SMD:C_0402_1005Metric, F.Cu at (-74.2, 174.5)
- added C25: 100nF, Capacitor_SMD:C_0402_1005Metric, F.Cu at (-74.2, 176.4)
- added R6: 2.5k, Resistor_SMD:R_0603_1608Metric, F.Cu at (-73.0, 173.9)
- added U10: STM32F405RGT6, Motor-Flasher:QFP50P1200X1200X160-64N, F.Cu at (126.0, 73.0)
- C1, C11, C14, C18, C2, C31, C32, C33, C34, C35, C7, R1, R10, R16, R2, R4, R5, R8: moved to F.Cu
- C10: value 4.7uF -> 100nF
- C19, C20: value 30pF -> 7pF; moved to F.Cu
- C8: value 1uF -> 2.2uF
- C9: value 4.7uF -> 2.2uF
- CR2: footprint smd110:SOD-123FL_MCC -> Motor-Flasher:SOD-123FL_MCC
- DS1: footprint revparts2:LCD_LCM-S01602DTR_A -> Motor-Flasher:LCD_LCM-S01602DTR_A
- J1: value USB4105-GF-A -> TYPE-C 16PIN 2MD(073); footprint revparts2:GCT_USB4105-GF-A -> Motor-Flasher:GCT_USB4105-GF-A
- J2: value Conn_01x04_MountingPin -> CS-1109-1X5(L11.5)PA6T; footprint Connector_PinHeader_2.54mm:PinHeader_1x04_P2.54mm_Horizontal -> Connector_PinHeader_2.54mm:PinHeader_1x05_P2.54mm_Horizontal
- J4: footprint revparts2:JST_B2B-XH-A -> Motor-Flasher:JST_B2B-XH-A
- J8: footprint revparts2:CUI_TB006-508-03BE -> Motor-Flasher:CUI_TB006-508-03BE
- L2: footprint revparts3:CDRH5D28RHP -> Motor-Flasher:CDRH5D28RHP
- PS5: footprint relevantparts:CONV_RFM-0505S -> Motor-Flasher:CONV_RFM-0505S
- R13: value 10k -> 220; moved to F.Cu
- R24, R26: value 10k -> 4.7k; moved to F.Cu
- R25: value 120 -> 4.7k; moved to F.Cu
- R9: value 10k -> 120
- S10, S11, S12, S13, S5: footprint revparts2:TS-1088-AR02016 -> Motor-Flasher:TS-1088-AR02016
- SW1, SW2, SW3, SW4: footprint revparts2:SS12D07_CNK -> Motor-Flasher:SS12D07_CNK
- SW5: footprint revparts2:SS12D07_CNK -> Motor-Flasher:SOT95P275X110-6N
- U1, U2, U4, U5: footprint revparts2:SOT95P275X110-6N -> Motor-Flasher:SOT95P275X110-6N; moved to F.Cu
- U19: footprint revparts2:SOIC127P1030X265-18N -> Motor-Flasher:SOIC127P1030X265-18N
- U20: footprint revparts2:SOP254P1040X485-8N -> Motor-Flasher:SOP254P1040X485-8N
- U3: footprint revparts2:SOT230P700X180-4N -> Motor-Flasher:SOT230P700X180-4N
- U6: footprint revparts2:VREG_V62_16624-01YE -> Motor-Flasher:VREG_V62_16624-01YE
- U9: footprint revparts2:SOIC127P1032X265-16N -> Motor-Flasher:SOIC127P1032X265-16N; moved to F.Cu
- VR1: footprint revparts3:POT_3362P -> Motor-Flasher:POT_3362P
- Y1: footprint RevParts:OSC_CSTNE16M0V530000R0 -> Motor-Flasher:OSC_CSTNE16M0V530000R0; moved to F.Cu
- Y2: footprint revparts2:OSC_CSTNE16M0V530000R0 -> Motor-Flasher:OSC_CSTNE16M0V530000R0
- moved L2 643.0 mm to (858.0, 238.0)
- moved SW4 516.9 mm to (-180.5, 429.5)
- moved VR1 466.0 mm to (-111.1, -328.0)
- moved Y1 450.0 mm to (-202.5, -186.5), turned to 0 degrees
- moved C19 441.4 mm to (-218.0, -150.5), turned to 0 degrees
- moved C20 429.0 mm to (-163.0, -206.0), turned to 0 degrees
- moved SW2 384.6 mm to (554.8, 74.0)
- moved J1 349.0 mm to (545.5, 183.0), turned to 90 degrees
- moved R7 345.5 mm to (581.0, 112.5), turned to 0 degrees
- moved C10 339.4 mm to (-77.0, 174.5)
- moved R3 335.9 mm to (578.6, 95.0), turned to 0 degrees
- moved C9 335.0 mm to (-77.0, 172.5), turned to 0 degrees
- moved C8 329.6 mm to (-77.0, 170.5), turned to 0 degrees
- moved R26 317.0 mm to (-71.3, 176.5)
- moved J4 312.2 mm to (552.8, 97.5), turned to 0 degrees
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Connections:
- net /LED/A renamed /LCD/A
- net /LED/D4L renamed /LCD/D4L
- net /LED/D5L renamed /LCD/D5L
- net /LED/D6L renamed /LCD/D6L
- net /LED/D7L renamed /LCD/D7L
- net /LED/E_L renamed /LCD/E_L
- net /LED/RS_L renamed /LCD/RS_L
- net /LED/RW_L renamed /LCD/RW_L
- C1 pad 1: VCC -> Vout
- C10 pad 1: Net-(U7-EN2) -> +3.3V
- C11 pad 1: +3.3V -> GND
- C11 pad 2: GND -> +3.3V
- C3 pad 1: VCC -> GND
- C3 pad 2: GND -> Vout
- C4 pad 1: VCC -> GND
- C4 pad 2: GND -> Vout
- C7 pad 1: GND -> /MCU/Boot0
- C7 pad 2: /MCU/Boot0 -> GND
- C8 pad 1: VDD -> Net-(U10-VCAP_1)
- C9 pad 1: VCC -> Net-(U10-VCAP_2)
- CR2 pad 1: Net-(CR2-Pad1) -> VDD
- J2 pad 1: +3.3V -> /MCU/Sys_CLK
- J2 pad 2: GND -> /MCU/Sys_SDIO
- J2 pad 3: /MCU/Sys_SDIO -> GND
- J2 pad 4: /MCU/Sys_CLK -> /MCU/NRST
- L2 pad 1: VCC -> Vout
- R24 pad 2: Net-(U23-~{RESET}) -> /SCL
- R25 pad 1: Net-(R25-Pad1) -> +3.3V
- R25 pad 2: /CAN3/CANL -> /SDA
- R26 pad 2: Net-(U25-~{RESET}) -> /LCD_Int
- R3 pad 1: VCC -> Vout
- R9 pad 1: GND -> Net-(R9-Pad1)
- R9 pad 2: Net-(U7-TS) -> /CAN1/CANL
- SW1 pad 2: Net-(R21-Pad1) -> Net-(R9-Pad1)
- SW2 pad 1: unconnected-(SW2-Pad1) -> VDD
- SW2 pad 2: Net-(R23-Pad1) -> Vout
- SW2 pad 3: /CAN2/CANH -> VCC
- SW3 pad 1: unconnected-(SW3-Pad1) -> /CAN1/CAN_TX
- SW3 pad 2: Net-(R25-Pad1) -> /CAN1/CANTX_OUT
- SW3 pad 3: /CAN3/CANH -> /CANTX
- SW4 pad 1: unconnected-(SW4-Pad1) -> /CAN1/CAN_RX
- SW4 pad 2: Net-(R27-Pad1) -> /CAN1/CANRX_OUT
- SW4 pad 3: /CAN4/CANH -> /CANRX
- U19 pad 12: /INT1 -> /INT
- U19 pad 16: /CS1 -> /CS
- U20 pad 2: /CAN1/CAN_RX -> /CAN1/CANRX_OUT
- U20 pad 3: /CAN1/CAN_TX -> /CAN1/CANTX_OUT
- U3 pad 3: VCC -> Vout
- U6 pad 1: VCC -> Vout
- U6 pad 6: VCC -> Vout
Routing:
- net +5V: track 274.0 -> 0.00 mm, vias 7 -> 0
- net GND: track 229.9 -> 0.00 mm, vias 59 -> 0
- net /SCK: track 141.0 -> 0.00 mm, vias 8 -> 0
- net /MISO: track 137.4 -> 0.00 mm, vias 5 -> 0
- net /MOSI: track 131.6 -> 0.00 mm, vias 4 -> 0
- net +3.3V: track 89.6 -> 0.00 mm, vias 12 -> 0
- net /CS4: track 69.5 -> 0.00 mm, vias 2 -> 0
- net /INT4: track 68.6 -> 0.00 mm
- net /D-: track 58.6 -> 0.00 mm, vias 1 -> 0
- net /D+: track 57.4 -> 0.00 mm, vias 1 -> 0
- net VCC: track 53.8 -> 0.00 mm, vias 6 -> 0
- net /INT1: track 51.2 -> 0.00 mm, vias 4 -> 0
- net /CS1: track 50.8 -> 0.00 mm, vias 2 -> 0
- net /SysOff: track 50.1 -> 0.00 mm
- net /MCU/Boot0: track 41.0 -> 0.00 mm, vias 3 -> 0
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- removed copper zone on B.Cu, net +3.3V
- removed copper zone on F.Cu, net +5V
- removed copper zone on F.Cu, net GND
- removed copper zone on F.Cu, net Net-(U7-EN2)
- removed copper zone on F.Cu, net VCC
- removed copper zone on F.Cu, net VDD
Other:
- board outline removed
- copper layers 2 -> 4
- board text removed: "Back"
- board text removed: "Boot"
- board text removed: "CANH"
- board text removed: "Down"
- board text removed: "High"
- board text removed: "Low"
- board text removed: "Off"
- board text removed: "Reset"
- board text removed: "Select"
- board text removed: "Up"

Commit message: Removed ERC Errors and Warnings
Parts:
- moved SW4 384.0 mm to (77.5, 145.1)
- moved U19 58.1 mm to (109.0, 131.1)
- moved C7 6.25 mm to (-75.5, 162.5)
Changed lines of the file:
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@@
 	(footprint "Capacitor_SMD:C_0402_1005Metric"
 		(layer "F.Cu")
-		(at -77.02 168.56)
+		(at -75.5 162.5)
 		(descr "Capacitor SMD 0402 (1005 Metric), square (rectangular) end terminal, IPC_7351 nominal, (Body size source: IPC-SM-782 page 76, https://www.pcb-3d.com/wordpress/wp-content/uploads/ipc-sm-782a_amendment_1_and_2.pdf), generated with kicad-footprint-generator")
 		(tags "capacitor")
@@
 		(at 176.77 246.25)
 		(property "Reference" "PS5"
-			(at -2.385 -4.745 360)
+			(at -2.385 -4.745 0)
 			(layer "F.SilkS")
 			(effects
@@
 		)
 		(property "Value" "B0505S-1WR3"
-			(at 3.08 4.295 360)
+			(at 3.08 4.295 0)
 			(layer "F.Fab")
 			(effects
@@
 		)
 		(property "Footprint" "Motor-Flasher:CONV_RFM-0505S"
-			(at 0 0 360)
+			(at 0 0 0)
 			(layer "F.Fab")
 			(hide yes)
@@
 		)
 		(property "Datasheet" ""
-			(at 0 0 360)
+			(at 0 0 0)
 			(layer "F.Fab")
 			(hide yes)
@@
 		)
 		(property "Description" ""
-			(at 0 0 360)
+			(at 0 0 0)
 			(layer "F.Fab")
 			(hide yes)
@@
 		)
 		(property "Footprint" "Motor-Flasher:SS12D07_CNK"
-			(at 0 0 360)
+			(at 0 0 0)
 			(layer "F.Fab")
 			(hide yes)
@@
 		)
 		(property "Datasheet" "SS12D07VG4NSGAPA"
-			(at 0 0 360)
+			(at 0 0 0)
 			(layer "F.Fab")
 			(hide yes)
@@
 		)
 		(property "Description" ""
-			(at 0 0 360)
+			(at 0 0 0)
 			(layer "F.Fab")
 			(hide yes)
@@
 		)
 		(fp_text user "*"
-			(at -2.6543 0 360)
+			(at -2.6543 0 0)
 			(layer "F.SilkS")
 			(effects
@@
 		)
 		(fp_text user "*"
-			(at -1.7653 0 360)
+			(at -1.7653 0 0)
 			(layer "F.Fab")
 			(effects
@@
 	(footprint "Motor-Flasher:SS12D07_CNK"
 		(layer "F.Cu")
-		(at -180.5 429.5)
+		(at 77.5 145.100001)
 		(tags "SS12D07VG4NSGAPA ")
 		(property "Reference" "SW4"
@@
 		)
 		(property "Footprint" "Motor-Flasher:SS12D07_CNK"
-			(at 0 0 360)
+			(at 0 0 0)
 			(layer "F.Fab")
 			(hide yes)
@@
 		)
 		(property "Datasheet" "SS12D07VG4NSGAPA"
-			(at 0 0 360)
+			(at 0 0 0)
 			(layer "F.Fab")
 			(hide yes)
@@
 		)
 		(property "Description" ""
-			(at 0 0 360)
+			(at 0 0 0)
 			(layer "F.Fab")
 			(hide yes)
@@
 		)
 		(fp_text user "*"
-			(at -2.6543 0 360)
+			(at -2.6543 0 0)
 			(layer "F.SilkS")
 			(effects
@@
 		)
 		(fp_text user "*"
-			(at -1.7653 0 360)
+			(at -1.7653 0 0)
 			(layer "F.Fab")
 			(effects
@@
 		(at 552.75 97.475)
 		(property "Reference" "J4"
-			(at 7.4173 56.7203 360)
+			(at 7.4173 56.7203 0)
 			(layer "F.SilkS")
 			(hide yes)
@@
 		)
 		(property "Value" "B2B-PH-K-S-GW"
-			(at 3.67 4.76 360)
+			(at 3.67 4.76 0)
 			(layer "F.Fab")
 			(effects
@@
 		)
 		(property "Footprint" "Motor-Flasher:JST_B2B-XH-A"
-			(at 0 0 360)
+			(at 0 0 0)
 			(layer "F.Fab")
 			(hide yes)
@@
 		)
 		(property "Datasheet" ""
-			(at 0 0 360)
+			(at 0 0 0)
 			(layer "F.Fab")
 			(hide yes)
@@
 		)
 		(property "Description" ""
-			(at 0 0 360)
+			(at 0 0 0)
 			(layer "F.Fab")
 			(hide yes)
@@
 		(at 126 73)
 		(property "Reference" "U10"
-			(at -2.613189 -8.47077 360)
+			(at -2.613189 -8.47077 0)
 			(layer "F.SilkS")
 			(effects
@@
 		)
 		(property "Value" "STM32F405RGT6"
-			(at 16.209365 8.578895 360)
+			(at 16.209365 8.578895 0)
 			(layer "F.Fab")
 			(hide yes)
@@
 		)
 		(property "Footprint" "Motor-Flasher:QFP50P1200X1200X160-64N"
-			(at 0 0 360)
+			(at 0 0 0)
 			(layer "F.Fab")
 			(hide yes)
@@
 		)
 		(property "Datasheet" ""
-			(at 0 0 360)
+			(at 0 0 0)
 			(layer "F.Fab")
 			(hide yes)
@@
 		)
 		(property "Description" ""
-			(at 0 0 360)
+			(at 0 0 0)
 			(layer "F.Fab")
 			(hide yes)
@@
 	(footprint "Motor-Flasher:SOIC127P1030X265-18N"
 		(layer "F.Cu")
-		(at 81 182 90)
+		(at 108.96 131.11 90)
 		(property "Reference" "U19"
 			(at -2.535 -6.637 90)

Commit message: Rough Placement and Design
Parts:
- removed C19, C20: 7pF, Capacitor_SMD:C_0402_1005Metric
- removed C31, C32: 7pF, Capacitor_SMD:C_0603_1608Metric
- removed CR2: SMD110PL-TP, Motor-Flasher:SOD-123FL_MCC
- removed DS1: HS1602A-B, Motor-Flasher:LCD_LCM-S01602DTR_A
- removed J1: TYPE-C 16PIN 2MD(073), Motor-Flasher:GCT_USB4105-GF-A
- removed J8: WJ500V-5.08-3P, Motor-Flasher:CUI_TB006-508-03BE
- removed L2: 6.8uH, Motor-Flasher:CDRH5D28RHP
- removed PS5: B0505S-1WR3, Motor-Flasher:CONV_RFM-0505S
- removed S10, S11, S12, S13, S5: TS-1088-AR02016, Motor-Flasher:TS-1088-AR02016
- removed SW1: SS12D07VG4NSGAPA, Motor-Flasher:SS12D07_CNK
- removed SW5: SS12D07VG4NSGAPA, Motor-Flasher:SOT95P275X110-6N
- removed U19: MCP2515-I_SO, Motor-Flasher:SOIC127P1030X265-18N
- removed U20: ISO1050DUBR, Motor-Flasher:SOP254P1040X485-8N
- added CR1: SMD110PL-TP, Motor-Flasher:SOD-123FL_MCC, F.Cu at (128.5, 85.0)
- added DS2: HS1602A-B, Motor-Flasher:LCD_LCM-S01602DTR_A, F.Cu at (103.5, 51.0)
- added J3: WJ500V-5.08-3P, Motor-Flasher:CUI_TB006-508-03BE, F.Cu at (98.0, 151.5)
- added J5: TYPE-C 16PIN 2MD(073), Motor-Flasher:GCT_USB4105-GF-A, F.Cu at (140.5, 83.0)
- added L1: 6.8uH, Motor-Flasher:CDRH5D28RHP, F.Cu at (78.5, 95.0)
- added PS1: B0505S-1WR3, Motor-Flasher:CONV_RFM-0505S, F.Cu at (100.0, 133.5)
- added S1: TS-1088-AR02016, Motor-Flasher:TS-1088-AR02016, F.Cu at (130.0, 73.5)
- added S2: TS-1088-AR02016, Motor-Flasher:TS-1088-AR02016, F.Cu at (109.0, 83.0)
- added S3: TS-1088-AR02016, Motor-Flasher:TS-1088-AR02016, F.Cu at (109.0, 79.0)
- added S4: TS-1088-AR02016, Motor-Flasher:TS-1088-AR02016, F.Cu at (109.0, 86.5)
- added S6: TS-1088-AR02016, Motor-Flasher:TS-1088-AR02016, F.Cu at (80.5, 84.0)
- added SW6: SS12D07VG4NSGAPA, Motor-Flasher:SS12D07_CNK, F.Cu at (106.0, 117.5)
- added SW7: SS12D07VG4NSGAPA, Motor-Flasher:SS12D07_CNK, F.Cu at (112.0, 117.5)
- added U7: MAX16054AZT_T, Motor-Flasher:SOT95P275X110-6N, F.Cu at (89.5, 85.0)
- added U8: STM32F405RGT6, Motor-Flasher:QFP50P1200X1200X160-64N, F.Cu at (98.0, 101.1)
- C3: value 10uF -> 2.2uF; footprint Capacitor_SMD:C_0805_2012Metric -> Capacitor_SMD:C_0402_1005Metric
- C4: value 100nF -> 47uF; footprint Capacitor_SMD:C_0402_1005Metric -> Capacitor_SMD:C_0805_2012Metric
- C5: value 2.2uF -> 10uF; footprint Capacitor_SMD:C_0402_1005Metric -> Capacitor_SMD:C_0805_2012Metric
- C6: value 47uF -> 100nF; footprint Capacitor_SMD:C_0805_2012Metric -> Capacitor_SMD:C_0402_1005Metric
- SW2: value SS12D07VG4NSGAPA -> SS12D07VG4NSGAPA_Powermux
- SW3: value SS12D07VG4NSGAPA -> SS12D07VG4NSGAPA_Boot
- SW4: value SS12D07VG4NSGAPA -> SS12D07VG4NSGAPA_120Ohms
- U10: value STM32F405RGT6 -> LD1117S33TR; footprint Motor-Flasher:QFP50P1200X1200X160-64N -> Motor-Flasher:SOT230P700X180-4N
- U3: value LD1117S33TR -> TPS61027DRCR; footprint Motor-Flasher:SOT230P700X180-4N -> Motor-Flasher:VREG_V62_16624-01YE
- U5: value MAX16054AZT_T -> MCP2515-I_SO; footprint Motor-Flasher:SOT95P275X110-6N -> Motor-Flasher:SOIC127P1030X265-18N
- U6: value TPS61027DRCR -> ISO1050DUBR; footprint Motor-Flasher:VREG_V62_16624-01YE -> Motor-Flasher:SOP254P1040X485-8N
- moved R3 508.6 mm to (70.0, 99.0)
- moved R7 508.5 mm to (73.0, 89.0), turned to 90 degrees
- moved VR1 438.7 mm to (63.5, 74.5)
- moved SW2 435.5 mm to (119.5, 88.9), turned to 180 degrees
- moved U6 423.6 mm to (113.5, 133.0), turned to -90 degrees
- moved U3 414.6 mm to (69.5, 94.5), turned to 0 degrees
- moved J4 412.8 mm to (140.0, 93.2), turned to 90 degrees
- moved Y1 405.9 mm to (87.5, 97.5), turned to -90 degrees
- moved R1 358.8 mm to (132.5, 81.5)
- moved R2 358.8 mm to (132.5, 83.5)
- moved R13 264.0 mm to (106.5, 71.0), turned to 90 degrees
- moved U5 236.2 mm to (94.7, 117.9), turned to 90 degrees
- moved C18 232.3 mm to (132.0, 75.0), turned to 90 degrees
- moved C14 229.8 mm to (85.0, 70.0)
- moved C11 227.2 mm to (90.5, 72.0), turned to 180 degrees
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Connections:
- C3 pad 1: GND -> +5V
- C3 pad 2: Vout -> GND
- C4 pad 1: GND -> +5V
- C4 pad 2: Vout -> GND
- C5 pad 1: +5V -> GND
- C5 pad 2: GND -> Vout
- C6 pad 1: +5V -> GND
- C6 pad 2: GND -> Vout
- C8 pad 1: Net-(U10-VCAP_1) -> Net-(U8-VCAP_1)
- C9 pad 1: Net-(U10-VCAP_2) -> Net-(U8-VCAP_2)
- R10 pad 2: Net-(U19-~{RESET}) -> Net-(U5-~{RESET})
- R3 pad 2: /USB + Power Source/LBI -> /Voltage Regulator/LBI
- R6 pad 1: Net-(U10-PB2/BOOT1) -> Net-(U8-PB2/BOOT1)
- R7 pad 1: /USB + Power Source/LBI -> /Voltage Regulator/LBI
- SW3 pad 1: /CAN1/CAN_TX -> GND
- SW3 pad 2: /CAN1/CANTX_OUT -> Net-(R8-Pad1)
- SW3 pad 3: /CANTX -> +3.3V
- SW4 pad 1: /CAN1/CAN_RX -> unconnected-(SW4-Pad1)
- SW4 pad 2: /CAN1/CANRX_OUT -> Net-(R9-Pad1)
- SW4 pad 3: /CANRX -> /CAN1/CANH
- U1 pad 1: /Buttons/Back -> /Buttons/Down
- U1 pad 5: /Deb_back -> /Deb_Down
- U10 pad 1: +3.3V -> GND
- U10 pad 2: unconnected-(U10-PC13/RTC_OUT-Pad2) -> +3.3V
- U10 pad 3: unconnected-(U10-PC14/OSC32_IN-Pad3) -> Vout
- U10 pad 4: unconnected-(U10-PC15/OSC32_OUT-Pad4) -> +3.3V
- U3 pad 1: GND -> Vout
- U3 pad 2: +3.3V -> +5V
- U3 pad 3: Vout -> unconnected-(U3-FB-Pad3)
- U3 pad 4: +3.3V -> unconnected-(U3-LBO-Pad4)
- U5 pad 1: /Buttons/Down -> /CAN1/CAN_TX
- U5 pad 2: GND -> /CAN1/CAN_RX
- U5 pad 3: GND -> unconnected-(U5-CLKOUT/SOF-Pad3)
- U5 pad 5: /Deb_Down -> unconnected-(U5-~{TX1RTS}-Pad5)
- U5 pad 6: +3.3V -> unconnected-(U5-~{TX2RTS}-Pad6)
- U6 pad 1: Vout -> +3.3V
- U6 pad 2: +5V -> /CAN1/CANRX_OUT
- U6 pad 3: unconnected-(U6-FB-Pad3) -> /CAN1/CANTX_OUT
- U6 pad 4: unconnected-(U6-LBO-Pad4) -> GND
- U6 pad 5: GND -> /CAN1/CAN_GND
- U6 pad 6: Vout -> /CAN1/CANL
- U6 pad 7: /USB + Power Source/LBI -> /CAN1/CANH
- U6 pad 8: GND -> /CAN1/CAN_VDD
- Y1 pad 1: /MCU/Osc1 -> /MCU/OscIn
- Y1 pad 3: /MCU/Osc2 -> /MCU/OscOut
Other:
- board outline added: 205.4 x 124.8 mm

Commit message: Saving current revision
Parts:
- moved S1 175.3 mm to (-43.8, 96.8)
- moved R16 175.3 mm to (-41.2, 98.5), turned to 90 degrees
- moved C18 174.4 mm to (-41.2, 94.9)
- moved R8 163.8 mm to (-39.4, 87.4), turned to -90 degrees
- moved SW3 162.9 mm to (-42.9, 90.2)
- moved C7 162.2 mm to (-37.7, 87.4), turned to 90 degrees
- moved Y1 119.2 mm to (-31.4, 89.6)
- moved C11 115.0 mm to (-22.9, 52.6), turned to -90 degrees
- moved U6 108.2 mm to (5.97, 120.5)
- moved R13 106.5 mm to (1.53, 53.2), turned to 0 degrees
- moved U8 105.2 mm to (-5.56, 82.7)
- moved R5 103.4 mm to (32.6, 53.1)
- moved C14 103.3 mm to (-16.6, 51.5)
- moved R1 103.2 mm to (32.4, 56.3)
- moved R2 103.2 mm to (32.5, 58.3)
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Connections:
- CR1 pad 1: VDD -> Vout
- CR1 pad 2: VBUS -> Net-(CR1-Pad2)
- J5 pad A4-B9: VBUS -> VDD
- J5 pad B4-A9: VBUS -> VDD
- SW2 pad 2: Vout -> Net-(CR1-Pad2)
Routing:
- net VDD: track 0.00 -> 7.22 mm
- net /USB + Power Source/USB_D+: track 0.00 -> 6.05 mm
- net /USB + Power Source/USB_D-: track 0.00 -> 5.77 mm
- net Net-(J5-CC1): track 0.00 -> 4.89 mm
- net Net-(J5-CC2): track 0.00 -> 4.26 mm
Other:
- board size 205.4 x 124.8 mm -> 83 x 124.8 mm
