File: InfineonController/mcu.kicad_sch (KiCad schematic)
At the start: 0 parts

Commit message: Current Changes pushed
Parts:
- added C1, C10, C11, C12, C13, C2, C3, C4, C5, C7, C8, C9: 100nF, symbol Device:C
- added C14, C15, C16, C17, C6: C, symbol Device:C
- added IC1: XMC4800F144F1024AAXQMA1, QFP50P2200X2200X160-144N, symbol XMC4800F144F1024AAXQMA1:XMC4800F144F1024AAXQMA1
- added Y1, Y2: Crystal, symbol Device:Crystal
Connections:
- new net VDDC: IC1.125 (VDDC_4), IC1.19 (VDDC_1), IC1.61 (VDDC_2), IC1.90 (VDDC_3)
- new net VDDP: IC1.126 (VDDP_4), IC1.18 (VDDP_1), IC1.62 (VDDP_2), IC1.86 (VDDP_3)
